File: pi_gps_tracker/PiZeroGPSHat.sch (EAGLE design)
At the start: 17 parts, among them IC1 24AA32ASM

Commit message: Added Jumper to WP.
Parts:
- removed TP1, TP2: TPB1,27, testpad:TPB1,27
- added JP1: (no value), pinhead:PINHD-1X2
Connections:
- removed net N$7: IC1.WP, R4.1, TP2.TP
- new net WP: IC1.WP, JP1.1, R4.1
- net GND: now also JP1.2; no longer TP1.TP
Changed lines of the file:
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@@
 <part name="R4" library="adafruit" deviceset="R-US_" device="R0805" value="9.9k"/>
 <part name="GND12" library="supply1" deviceset="GND" device=""/>
-<part name="TP1" library="testpad" deviceset="TP" device="B1,27"/>
-<part name="TP2" library="testpad" deviceset="TP" device="B1,27"/>
 <part name="TP3" library="testpad" deviceset="TP" device="B1,27"/>
 <part name="TP4" library="testpad" deviceset="TP" device="B1,27"/>
 <part name="TP5" library="testpad" deviceset="TP" device="B1,27"/>
 <part name="TP6" library="testpad" deviceset="TP" device="B1,27"/>
+<part name="JP1" library="pinhead" deviceset="PINHD-1X2" device=""/>
 </parts>
 <sheets>
@@
 <instance part="R4" gate="G$1" x="40.64" y="88.9" rot="R90"/>
 <instance part="GND12" gate="1" x="12.7" y="81.28" rot="R270"/>
-<instance part="TP1" gate="G$1" x="22.86" y="81.28" rot="R270"/>
-<instance part="TP2" gate="G$1" x="30.48" y="81.28" rot="R90"/>
 <instance part="TP3" gate="G$1" x="63.5" y="45.72" rot="R90"/>
 <instance part="TP4" gate="G$1" x="167.64" y="33.02" rot="R270"/>
 <instance part="TP5" gate="G$1" x="160.02" y="30.48" rot="R270"/>
 <instance part="TP6" gate="G$1" x="20.32" y="-15.24" rot="R180"/>
+<instance part="JP1" gate="G$1" x="27.94" y="88.9"/>
 </instances>
 <busses>
@@
 <pinref part="GND12" gate="1" pin="GND"/>
 <wire x1="20.32" y1="81.28" x2="15.24" y2="81.28" width="0.1524" layer="91"/>
-<pinref part="TP1" gate="G$1" pin="TP"/>
+<wire x1="20.32" y1="81.28" x2="20.32" y2="88.9" width="0.1524" layer="91"/>
+<pinref part="JP1" gate="G$1" pin="2"/>
+<wire x1="20.32" y1="88.9" x2="25.4" y2="88.9" width="0.1524" layer="91"/>
 </segment>
 </net>
@@
 </segment>
 </net>
-<net name="N$7" class="0">
+<net name="WP" class="0">
 <segment>
 <wire x1="33.02" y1="81.28" x2="40.64" y2="81.28" width="0.1524" layer="91"/>
@@
 <wire x1="40.64" y1="83.82" x2="40.64" y2="81.28" width="0.1524" layer="91"/>
 <junction x="40.64" y="81.28"/>
-<pinref part="TP2" gate="G$1" pin="TP"/>
-</segment>
-</net>
+<pinref part="JP1" gate="G$1" pin="1"/>
+<wire x1="25.4" y1="91.44" x2="33.02" y2="91.44" width="0.1524" layer="91"/>
+<wire x1="33.02" y1="91.44" x2="33.02" y2="81.28" width="0.1524" layer="91"/>
+</segment>
+</net>

Commit message: V2 of the GPS hat to add LEDs for status indicators
Parts:
- added LED2, LED3: 1, adafruit:LEDCHIPLED_0805
- added R5, R6: 470, adafruit:R-US_R0805
Connections:
- removed net N$3: TP5.TP, U1.1PPS
- new net 1PPS: LED3.A, TP5.TP, U1.1PPS
- new net N$7: LED2.C, R5.2
- new net N$8: LED3.C, R6.2
- net +3V3: now also LED2.A
- net GND: now also R5.1, R6.1
Changed lines of the file:
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@@
 <?xml version="1.0" encoding="utf-8"?>
 <!DOCTYPE eagle SYSTEM "eagle.dtd">
-<eagle version="7.3.0">
+<eagle version="7.5.0">
 <drawing>
 <settings>
@@
 <part name="TP6" library="testpad" deviceset="TP" device="B1,27"/>
 <part name="JP1" library="pinhead" deviceset="PINHD-1X2" device=""/>
+<part name="LED2" library="adafruit" deviceset="LED" device="CHIPLED_0805" value="1"/>
+<part name="R5" library="adafruit" deviceset="R-US_" device="R0805" value="470"/>
+<part name="GND13" library="supply1" deviceset="GND" device=""/>
+<part name="LED3" library="adafruit" deviceset="LED" device="CHIPLED_0805" value="1"/>
+<part name="R6" library="adafruit" deviceset="R-US_" device="R0805" value="470"/>
+<part name="GND14" library="supply1" deviceset="GND" device=""/>
 </parts>
 <sheets>
@@
 <instance part="TP6" gate="G$1" x="20.32" y="-15.24" rot="R180"/>
 <instance part="JP1" gate="G$1" x="27.94" y="88.9"/>
+<instance part="LED2" gate="G$1" x="137.16" y="76.2" rot="R270"/>
+<instance part="R5" gate="G$1" x="121.92" y="76.2"/>
+<instance part="GND13" gate="1" x="114.3" y="76.2" rot="R270"/>
+<instance part="LED3" gate="G$1" x="152.4" y="63.5" rot="R270"/>
+<instance part="R6" gate="G$1" x="142.24" y="63.5"/>
+<instance part="GND14" gate="1" x="134.62" y="63.5" rot="R270"/>
 </instances>
 <busses>
@@
 <wire x1="20.32" y1="88.9" x2="25.4" y2="88.9" width="0.1524" layer="91"/>
 </segment>
+<segment>
+<pinref part="R5" gate="G$1" pin="1"/>
+<pinref part="GND13" gate="1" pin="GND"/>
+</segment>
+<segment>
+<pinref part="R6" gate="G$1" pin="1"/>
+<pinref part="GND14" gate="1" pin="GND"/>
+</segment>
 </net>
 <net name="UART0_TXD" class="0">
@@
 </segment>
 </net>
-<net name="N$3" class="0">
+<net name="1PPS" class="0">
 <segment>
 <pinref part="U1" gate="G$1" pin="1PPS"/>
 <wire x1="137.16" y1="30.48" x2="157.48" y2="30.48" width="0.1524" layer="91"/>
 <pinref part="TP5" gate="G$1" pin="TP"/>
+<label x="152.4" y="30.48" size="1.778" layer="95"/>
+</segment>
+<segment>
+<pinref part="LED3" gate="G$1" pin="A"/>
+<wire x1="154.94" y1="63.5" x2="167.64" y2="63.5" width="0.1524" layer="91"/>
+<label x="162.56" y="63.5" size="1.778" layer="95"/>
 </segment>
 </net>
@@
 <junction x="40.64" y="111.76"/>
 </segment>
+<segment>
+<pinref part="LED2" gate="G$1" pin="A"/>
+<wire x1="139.7" y1="76.2" x2="152.4" y2="76.2" width="0.1524" layer="91"/>
+<label x="149.86" y="76.2" size="1.778" layer="95"/>
+</segment>
 </net>
 <net name="N$5" class="0">
@@
 </segment>
 </net>
+<net name="N$7" class="0">
+<segment>
+<pinref part="LED2" gate="G$1" pin="C"/>
+<pinref part="R5" gate="G$1" pin="2"/>
+<wire x1="132.08" y1="76.2" x2="127" y2="76.2" width="0.1524" layer="91"/>
+</segment>
+</net>
+<net name="N$8" class="0">
+<segment>
+<pinref part="LED3" gate="G$1" pin="C"/>
+<pinref part="R6" gate="G$1" pin="2"/>
+</segment>
+</net>

Commit message: V3 moved all the LEDs to the same location.
Parts:
- renumbered LED1 to _
Changed lines of the file:
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@@
 <part name="R1" library="adafruit" deviceset="R-US_" device="R0805" value="9.9k"/>
 <part name="R2" library="adafruit" deviceset="R-US_" device="R0805" value="470"/>
-<part name="LED1" library="adafruit" deviceset="LED" device="CHIPLED_0805" value="1"/>
+<part name="_" library="adafruit" deviceset="LED" device="CHIPLED_0805" value="1"/>
 <part name="IC1" library="microchip" deviceset="24*" device="SM" technology="AA32A"/>
 <part name="C1" library="resistor" deviceset="C-US" device="C0402" value="0.1uF"/>
@@
 <instance part="R1" gate="G$1" x="35.56" y="106.68" rot="R90"/>
 <instance part="R2" gate="G$1" x="68.58" y="38.1"/>
-<instance part="LED1" gate="G$1" x="81.28" y="38.1" rot="R270"/>
+<instance part="_" gate="G$1" x="81.28" y="38.1" rot="R270"/>
 <instance part="IC1" gate="G$1" x="71.12" y="88.9"/>
 <instance part="C1" gate="G$1" x="91.44" y="55.88"/>
@@
 <segment>
 <pinref part="U1" gate="G$1" pin="3D-FIX"/>
-<pinref part="LED1" gate="G$1" pin="A"/>
+<pinref part="_" gate="G$1" pin="A"/>
 <wire x1="106.68" y1="38.1" x2="83.82" y2="38.1" width="0.1524" layer="91"/>
 </segment>
@@
 <net name="N$2" class="0">
 <segment>
-<pinref part="LED1" gate="G$1" pin="C"/>
+<pinref part="_" gate="G$1" pin="C"/>
 <pinref part="R2" gate="G$1" pin="2"/>
 <wire x1="76.2" y1="38.1" x2="73.66" y2="38.1" width="0.1524" layer="91"/>

Commit message: New Board and SCAD
Parts:
- removed D1: ES2D, diode:ES2D
- removed TP6: TPB1,27, testpad:TPB1,27
- added LED1: 1, adafruit:LEDCHIPLED_0805
- added R7: 470, adafruit:R-US_R0402
- R1, R3: value 9.9k -> 3.9k; device adafruit:R-US_R0805 -> adafruit:R-US_R0402
- R2, R5, R6: device adafruit:R-US_R0805 -> adafruit:R-US_R0402
- R4: value 9.9k -> 1.2k; device adafruit:R-US_R0805 -> adafruit:R-US_R0402
- renumbered LED2 to 3V3, LED3 to 1PPS, _ to FIX
Connections:
- removed net +5V: R.2, R.4, TP6.TP
- new net GP2: R.3
- new net GP3: R.5
- new net GP4: LED1.A, R.7
- new net N$3: LED1.C, R7.2
- net GND: now also R7.1; no longer D1.C
- net N$6: no longer D1.A
